Commit message: remove radar plugin in bolt

File: final_project/catkin_ws/src/car_demo/bolt_description/urdf/bolt.urdf (robot description, URDF)
Before this commit: robot bolt, 28 links, 27 joints
Joints:
- removed joint radar_joint

Commit message: fix car reposition problem by removing radar plugin

File: final_project/catkin_ws/src/car_demo/bolt_description/urdf/bolt.urdf (robot description, URDF)
Before this commit: robot bolt, 28 links, 26 joints
Links:
- removed link rad_link
